File: LeachAmp_kicad/LeachAmp_kicad.kicad_pcb (KiCad board)
At the start: 2 copper layers, 117 parts, among them J1 Conn_01x04_Male, J2 Conn_01x02_Male, J3 Conn_01x03_Female, Q1 BC546, Q10 MPSA06, Q11 MPSA56, Q12 BF470, Q13 BF469, Q14 BF469, Q15 BF470, Q16 MJE15030, Q17 MJE15031, Q2 BC546, Q3 BC556, Q4 BC556, Q5 BC546, Q6 BC556, Q7 BD139, Q8 BC556, Q9 BC546, T1 MJL3281, T2 MJL3201, T3 MJL3281, T4 MJL3201

Commit message: Schéma komplet + DPS v progresu
Kompletní schéma Leach verze.
DPS rozpracované - silová část
Parts:
- added REF**: MountingHole_3.2mm_M3_DIN965_Pad, MountingHole:MountingHole_3.2mm_M3_DIN965_Pad, F.Cu at (209.3, 45.3)
- added REF**: MountingHole_3.2mm_M3_DIN965_Pad, MountingHole:MountingHole_3.2mm_M3_DIN965_Pad, F.Cu at (120.0, 45.3)
- added REF**: MountingHole_3.2mm_M3_DIN965_Pad, MountingHole:MountingHole_3.2mm_M3_DIN965_Pad, F.Cu at (209.3, 137.6)
- added REF**: MountingHole_3.2mm_M3_DIN965_Pad, MountingHole:MountingHole_3.2mm_M3_DIN965_Pad, F.Cu at (120.0, 137.6)
- F1, F2: footprint Fuse:Fuseholder_Cylinder-5x20mm_Schurter_0031_8201_Horizontal_Open -> Fuse_Holders_and_Fuses:Fuseholder5x20_horiz_SemiClosed_Casing10x25mm
- J1: value Conn_01x04_Male -> Conn_01x12_Female; footprint Connector_Wago:Wago_734-164_1x04_P3.50mm_Horizontal -> LeachAmp_library:Wago-256-406
- J2: value Conn_01x02_Male -> Conn_01x04_Female; footprint Connector_Wago:Wago_734-162_1x02_P3.50mm_Horizontal -> LeachAmp_library:Wago-256-402
- moved C1 235.1 mm to (-112.8, 114.8)
- moved C10 235.1 mm to (-49.6, 104.8)
- moved C11 235.1 mm to (6.11, 49.3)
- moved C12 235.1 mm to (-45.0, 100.0)
- moved C14 235.1 mm to (-25.0, 18.9)
- moved C15 235.1 mm to (-5.14, 45.8)
- moved C16 235.1 mm to (-18.4, 57.3)
- moved C2 235.1 mm to (-5.14, 53.0)
- moved C24 235.1 mm to (7.24, 35.8)
- moved C27 235.1 mm to (-37.4, 81.0)
- moved C3 235.1 mm to (-72.8, 113.7)
- moved C5 235.1 mm to (-100.4, 109.0)
- moved C6A1 235.1 mm to (-59.4, 108.5)
- moved C6B1 235.1 mm to (-22.7, 74.0)
- moved C7 235.1 mm to (-61.3, 116.8)
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Connections:
- J1 pad 1: +VCC -> -VCC
- J1 pad 2: GND -> -VCC
- J1 pad 4: Net-(J1-Pad4) -> -VCC
- J2 pad 2: GND -> out
Routing:
- net GND: track 0.00 -> 191.2 mm
- net Net-(C17-Pad1): track 0.00 -> 173.8 mm, vias 0 -> 1
- net +VCC: track 0.00 -> 70.8 mm, vias 1 -> 0
- net -VCC: track 0.00 -> 70.7 mm, vias 1 -> 0
- net Net-(C20-Pad2): track 0.00 -> 63.2 mm
- net Net-(Q16-Pad1): track 0.00 -> 57.2 mm
- net Net-(C24-Pad1): track 0.00 -> 57.1 mm
- net Net-(C19-Pad1): track 0.00 -> 54.8 mm
- net Net-(C18-Pad1): track 0.00 -> 50.5 mm
- net Net-(C17-Pad2): track 0.00 -> 49.8 mm
- net Net-(C23-Pad2): track 0.00 -> 46.5 mm
- net Net-(Q17-Pad1): track 0.00 -> 44.2 mm
- net Net-(R38-Pad1): track 0.00 -> 27.4 mm
- net Net-(R37-Pad1): track 0.00 -> 20.4 mm
- net out: track 0.00 -> 17.5 mm
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- added copper zone on B.Cu, net +VCC
- added copper zone on B.Cu, net -VCC
- added copper zone on F.Cu, net GND
- added copper zone on B.Cu, net out
Other:
- board outline added: 269.7 x 104.9 mm

Commit message: DPS progress 70%
DPS z většiny zpracovaná:
Výkonová část 85 %;
signální 60 %;
zpětná vazba 20 %.
Parts:
- added J4: Conn_01x03_Female, Connector_Molex:Molex_KK-254_AE-6410-03A_1x03_P2.54mm_Vertical, F.Cu at (110.9, 88.9)
- added REF**: MountingHole_3.2mm_M3_DIN965_Pad, MountingHole:MountingHole_3.2mm_M3_DIN965_Pad, F.Cu at (66.6, 45.3)
- added REF**: MountingHole_3.2mm_M3_DIN965_Pad, MountingHole:MountingHole_3.2mm_M3_DIN965_Pad, F.Cu at (66.6, 137.6)
- added REF**: MountingHole_3.2mm_M3_DIN965_Pad, MountingHole:MountingHole_3.2mm_M3_DIN965_Pad, F.Cu at (324.3, 137.6)
- added REF**: MountingHole_3.2mm_M3_DIN965_Pad, MountingHole:MountingHole_3.2mm_M3_DIN965_Pad, F.Cu at (324.3, 45.3)
- Q12, Q13: footprint Package_TO_SOT_THT:TO-126-3_Horizontal_TabDown -> Package_TO_SOT_THT:TO-126-3_Vertical
- moved R32 260.8 mm to (126.0, 54.6), turned to 180 degrees
- moved D5 251.3 mm to (148.2, 78.9), turned to 180 degrees
- moved D6 226.1 mm to (138.0, 104.0)
- moved C23 221.5 mm to (202.4, 69.0), turned to 270 degrees
- moved C6 220.8 mm to (177.0, 69.0), turned to 270 degrees
- moved R33 220.3 mm to (106.8, 127.3)
- moved D15 211.3 mm to (82.4, 147.4)
- moved C27 195.5 mm to (154.9, 116.0), turned to 90 degrees
- moved C5 193.8 mm to (93.1, 120.3), turned to 90 degrees
- moved C12 188.9 mm to (101.3, 219.5)
- moved C24 187.7 mm to (180.3, 108.3), turned to 270 degrees
- moved R15 186.0 mm to (90.0, 57.9)
- moved R20 185.9 mm to (148.6, 23.0)
- moved C10 180.4 mm to (126.7, 66.9)
- moved C14 179.0 mm to (106.8, 140.1), turned to 90 degrees
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Connections:
- Q7 pad 1: Net-(C11-Pad1) -> Net-(Q7-Pad1)
- Q7 pad 3: Net-(C10-Pad1) -> Net-(Q7-Pad3)
- R25 pad 1: Net-(Q7-Pad2) -> Net-(J4-Pad2)
- R27 pad 1: Net-(Q7-Pad2) -> Net-(J4-Pad2)
Routing:
- net GND: track 191.2 -> 778.5 mm, vias 0 -> 4
- net Net-(C24-Pad1): track 57.1 -> 210.9 mm
- net Net-(C23-Pad2): track 46.5 -> 188.5 mm
- net Net-(R20-Pad1): track 0.00 -> 55.5 mm
- net Net-(Q17-Pad1): track 44.2 -> 71.8 mm
- net Net-(Q14-Pad1): track 0.00 -> 25.7 mm
- net Net-(Q16-Pad1): track 57.2 -> 82.9 mm
- net Net-(Q15-Pad1): track 0.00 -> 21.7 mm
- net out: track 17.5 -> 35.2 mm
- net Net-(C10-Pad1): track 0.00 -> 13.9 mm
- net +VCC: track 70.8 -> 81.5 mm
- net Net-(R44-Pad2): track 0.00 -> 10.6 mm
- net Net-(C11-Pad1): track 0.00 -> 10.5 mm
- net Net-(C9-Pad1): track 0.00 -> 9.52 mm
- net Net-(D6-Pad1): track 0.00 -> 8.58 mm
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
Commit message: DPS progress 90 %
DPS z většiny zpracovaná:
Výkonová část 85 %;
signální 80 %;
zpětná vazba 40 %.
Parts:
- removed C12: 100n/50V film, Capacitor_THT:C_Rect_L7.2mm_W3.5mm_P5.00mm_FKS2_FKP2_MKS2_MKP2
- removed Q7: BD139, Package_TO_SOT_THT:TO-92_Inline
- moved R24 188.7 mm to (113.7, 114.9)
- moved R22 185.8 mm to (113.7, 120.1)
- moved R27 177.7 mm to (105.7, 114.7), turned to 90 degrees
- moved R25 146.7 mm to (100.8, 114.7), turned to 90 degrees
- moved R17 143.3 mm to (119.3, 74.5), turned to 180 degrees
- moved C8 96.8 mm to (105.3, 78.2), turned to 270 degrees
- moved C1 27.7 mm to (64.1, 114.0)
- moved D13 18.1 mm to (82.4, 53.3), turned to 90 degrees
- moved C2 17.6 mm to (89.2, 58.4)
- moved C6A1 16.7 mm to (98.2, 99.7), turned to 90 degrees
- moved C6B1 16.0 mm to (98.2, 83.2), turned to 270 degrees
- moved C15 15.4 mm to (95.2, 43.2)
- moved C16 15.1 mm to (95.5, 132.1)
- moved D14 15.0 mm to (88.0, 53.5), turned to 90 degrees
- moved C3 14.7 mm to (89.5, 125.7)
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Routing:
- net GND: track 778.5 -> 1561.7 mm
- net Net-(C14-Pad2): track 0.00 -> 71.9 mm
- net GNDS: track 0.00 -> 65.7 mm, vias 0 -> 2
- net Net-(C3-Pad2): track 0.00 -> 55.7 mm
- net Net-(C17-Pad1): track 177.7 -> 152.0 mm
- net Net-(C24-Pad1): track 210.9 -> 186.3 mm
- net Net-(C23-Pad2): track 188.5 -> 167.9 mm
- net Net-(C6A1-Pad1): track 0.00 -> 19.1 mm
- net Net-(C18-Pad1): track 56.4 -> 40.9 mm
- net Net-(C17-Pad2): track 55.2 -> 40.5 mm
- net Net-(D13-Pad2): track 0.00 -> 12.6 mm
- net Net-(D15-Pad1): track 0.00 -> 12.3 mm
- net Net-(C11-Pad2): track 6.10 -> 17.5 mm
- net Net-(C6A1-Pad2): track 0.00 -> 6.51 mm
- net Net-(Q3-Pad1): track 0.00 -> 5.72 mm
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Other:
- outline, holes or cut-outs redrawn

Commit message: DPS 100%
Parts:
- moved C9 53.5 mm to (99.8, 74.5)
- moved R20 52.3 mm to (127.6, 70.9), turned to 180 degrees
- moved R1 10.6 mm to (65.7, 97.8), turned to 270 degrees
- moved R23 10.2 mm to (113.7, 66.2), turned to 0 degrees
- moved R2 8.98 mm to (65.7, 85.2)
- moved R11 5.47 mm to (77.0, 51.4)
- moved R13 4.07 mm to (72.1, 51.4)
- moved C10 3.69 mm to (130.4, 66.8)
- moved R34 3.56 mm to (148.3, 66.8)
- moved C1 3.29 mm to (65.7, 111.1), turned to 270 degrees
- moved R32 2.42 mm to (123.8, 56.4)
- moved D8 1.55 mm to (116.3, 107.1)
- moved R33 1.40 mm to (113.7, 126.5)
- moved D7 0.81 mm to (109.7, 79.2)
- moved RV1 0.77 mm to (113.9, 98.6)
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Routing:
- net GND: track 1561.7 -> 2025.4 mm, vias 4 -> 6
- net Net-(C13-Pad1): track 0.00 -> 89.1 mm
- net Net-(C2-Pad2): track 0.00 -> 84.1 mm
- net Net-(C10-Pad2): track 6.23 -> 77.0 mm
- net Net-(C11-Pad2): track 17.5 -> 77.6 mm
- net Net-(C10-Pad1): track 13.9 -> 72.8 mm
- net Net-(Q9-Pad2): track 0.00 -> 47.5 mm
- net Net-(Q8-Pad2): track 0.00 -> 46.9 mm
- net GNDS: track 65.7 -> 108.4 mm
- net Net-(C1-Pad2): track 4.83 -> 45.9 mm
- net Net-(C17-Pad1): track 152.0 -> 191.9 mm
- net Net-(C11-Pad1): track 10.5 -> 50.0 mm
- net Net-(J4-Pad2): track 0.00 -> 32.5 mm
- net Net-(C24-Pad1): track 186.3 -> 217.1 mm
- net Net-(C3-Pad2): track 55.7 -> 84.5 mm
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
Commit message: DPS dokončeno
Parts:
- removed REF** (x8): MountingHole_3.2mm_M3_DIN965_Pad, MountingHole:MountingHole_3.2mm_M3_DIN965_Pad
- added  : MountingHole_3.2mm_M3_DIN965_Pad, MountingHole:MountingHole_3.2mm_M3_DIN965_Pad, F.Cu at (77.6, 45.3)
- added  : MountingHole_3.2mm_M3_DIN965_Pad, MountingHole:MountingHole_3.2mm_M3_DIN965_Pad, F.Cu at (77.6, 137.6)
- added  : MountingHole_3.2mm_M3_DIN965_Pad, MountingHole:MountingHole_3.2mm_M3_DIN965_Pad, F.Cu at (328.0, 137.6)
- added  : MountingHole_3.2mm_M3_DIN965_Pad, MountingHole:MountingHole_3.2mm_M3_DIN965_Pad, F.Cu at (328.0, 45.3)
- added  : MountingHole_3.2mm_M3_DIN965_Pad, MountingHole:MountingHole_3.2mm_M3_DIN965_Pad, F.Cu at (220.3, 45.3)
- added  : MountingHole_3.2mm_M3_DIN965_Pad, MountingHole:MountingHole_3.2mm_M3_DIN965_Pad, F.Cu at (131.0, 45.3)
- added  : MountingHole_3.2mm_M3_DIN965_Pad, MountingHole:MountingHole_3.2mm_M3_DIN965_Pad, F.Cu at (220.3, 137.6)
- added  : MountingHole_3.2mm_M3_DIN965_Pad, MountingHole:MountingHole_3.2mm_M3_DIN965_Pad, F.Cu at (131.0, 137.6)
- J1: value Conn_01x12_Female -> (none)
- J2: value Conn_01x04_Female -> (none)
- moved D15 11.1 mm to (93.5, 139.7)
- moved C17 11.0 mm to (135.8, 85.6)
- moved C18 11.0 mm to (135.8, 102.2)
- moved C1 11.0 mm to (76.7, 111.1)
- moved C10 11.0 mm to (141.4, 66.8)
- moved C11 11.0 mm to (142.8, 116.0)
- moved C13 11.0 mm to (117.8, 43.2)
- moved C14 11.0 mm to (117.8, 132.1)
- moved C15 11.0 mm to (106.2, 43.2)
- moved C16 11.0 mm to (106.5, 132.1)
- moved C19 11.0 mm to (157.3, 88.1)
- moved C2 11.0 mm to (100.2, 58.4)
- moved C20 11.0 mm to (157.3, 99.6)
- moved C21 11.0 mm to (313.5, 67.6)
- moved C22 11.0 mm to (275.9, 105.2)
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Other:
- board size 269.7 x 104.9 mm -> 262.4 x 104.9 mm

Commit message: Kondenzatory v prostred
Parts:
- removed the   at (220.3, 45.3)
- removed the   at (220.3, 137.6)
- added C12: 100n/50V film, Capacitor_THT:C_Rect_L7.2mm_W3.5mm_P5.00mm_FKS2_FKP2_MKS2_MKP2, F.Cu at (440.8, 167.4)
- added C28: CP, Capacitor_THT:CP_Radial_D25.0mm_P10.00mm_SnapIn, F.Cu at (176.2, 113.1)
- added C29: CP, Capacitor_THT:CP_Radial_D25.0mm_P10.00mm_SnapIn, F.Cu at (176.2, 139.1)
- added C30: CP, Capacitor_THT:CP_Radial_D25.0mm_P10.00mm_SnapIn, F.Cu at (233.5, 113.1)
- added C31: CP, Capacitor_THT:CP_Radial_D25.0mm_P10.00mm_SnapIn, F.Cu at (207.5, 139.1)
- added C32: CP, Capacitor_THT:CP_Radial_D25.0mm_P10.00mm_SnapIn, F.Cu at (323.6, 94.2)
- added C33: CP, Capacitor_THT:CP_Radial_D25.0mm_P10.00mm_SnapIn, F.Cu at (207.5, 113.1)
- added C34: CP, Capacitor_THT:CP_Radial_D25.0mm_P10.00mm_SnapIn, F.Cu at (350.9, 67.6)
- added C35: CP, Capacitor_THT:CP_Radial_D25.0mm_P10.00mm_SnapIn, F.Cu at (350.9, 94.2)
- added J5: Conn_01x03_Female, Connector_Molex:Molex_KK-254_AE-6410-03A_1x03_P2.54mm_Vertical, F.Cu at (431.6, 168.9)
- added Q7: BD139, Package_TO_SOT_THT:TO-92_Inline, F.Cu at (431.2, 176.0)
- C21, C22, C25, C26: footprint Capacitor_THT:CP_Radial_D35.0mm_P10.00mm_SnapIn -> Capacitor_THT:CP_Radial_D25.0mm_P10.00mm_SnapIn
- J1: value (none) -> Conn_01x12_Female
- J2: value (none) -> Conn_01x04_Female
- moved C21 169.6 mm to (150.2, 113.1)
- moved C25 166.8 mm to (150.2, 139.1)
- moved R43 128.8 mm to (278.2, 158.1)
- moved J1 126.7 mm to (126.1, 143.4)
- moved F1 69.7 mm to (191.8, 109.1), turned to 90 degrees
- moved R48 69.4 mm to (220.7, 169.7), turned to 0 degrees
- moved R46 69.2 mm to (220.7, 161.7), turned to 0 degrees
- moved F2 68.9 mm to (191.8, 153.1), turned to 270 degrees
- moved C27 68.0 mm to (201.9, 173.6)
- moved R42 66.5 mm to (199.8, 178.8)
- moved   65.6 mm to (380.0, 177.6)
- moved   65.6 mm to (380.0, 85.3)
- moved R45 64.9 mm to (241.0, 100.8), turned to 180 degrees
- moved R29 64.8 mm to (90.2, 134.2)
- moved C1 64.8 mm to (25.7, 151.1)
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Routing:
- net GND: track 2025.4 -> 1049.1 mm, vias 6 -> 1
- net Net-(C23-Pad2): track 195.9 -> 149.4 mm
- net Net-(Q16-Pad1): track 82.9 -> 42.0 mm
- net Net-(C17-Pad1): track 191.9 -> 151.6 mm
- net -VCC: track 78.4 -> 109.3 mm
- net +VCC: track 81.5 -> 108.8 mm
- net Net-(C24-Pad1): track 217.1 -> 195.3 mm
- net Net-(R38-Pad1): track 29.8 -> 50.0 mm
- net Net-(R43-Pad2): track 16.3 -> 0.00 mm
- net Net-(R41-Pad2): track 16.2 -> 0.00 mm
- net Net-(C20-Pad2): track 64.2 -> 51.0 mm
- net Net-(R42-Pad2): track 10.6 -> 21.0 mm
- net Net-(R44-Pad2): track 10.6 -> 20.9 mm
- net Net-(C18-Pad1): track 55.3 -> 45.4 mm
- net Net-(R37-Pad1): track 21.2 -> 31.0 mm
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- added copper zone on B.Cu, net GND
- removed copper zone on F.Cu, net GND
Other:
- board size 262.4 x 104.9 mm -> 365.4 x 104.9 mm

Commit message: Opraveny Tranzistory
Opraveny Tranzistory
Parts:
- removed C12: 100n/50V film, Capacitor_THT:C_Rect_L7.2mm_W3.5mm_P5.00mm_FKS2_FKP2_MKS2_MKP2
- removed C26, C32, C34, C35: CP, Capacitor_THT:CP_Radial_D25.0mm_P10.00mm_SnapIn
- removed J5: Conn_01x03_Female, Connector_Molex:Molex_KK-254_AE-6410-03A_1x03_P2.54mm_Vertical
- removed Q7: BD139, Package_TO_SOT_THT:TO-92_Inline
- T2, T4: value MJL3201 -> MJL1302
- moved R43 107.6 mm to (202.1, 82.0), turned to 270 degrees
- moved R44 44.7 mm to (213.0, 181.0), turned to 90 degrees
- moved R41 31.8 mm to (170.8, 82.0), turned to 270 degrees
- moved T4 31.4 mm to (212.9, 161.4)
- moved T2 31.4 mm to (181.4, 161.3)
- moved T1 31.3 mm to (170.8, 101.0)
- moved T3 31.3 mm to (202.1, 101.0)
- moved R42 18.4 mm to (181.5, 180.9), turned to 90 degrees
- moved R46 9.30 mm to (220.7, 171.0)
- moved R47 7.60 mm to (241.1, 100.3)
- moved R48 7.60 mm to (220.7, 162.1)
- moved R45 7.50 mm to (241.1, 93.3)
- moved C27 5.89 mm to (207.6, 175.1)
- moved C24 5.60 mm to (176.0, 167.6)
- moved C6 5.59 mm to (176.2, 88.0)
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Connections:
- T1 pad 2: Net-(R37-Pad1) -> Net-(C23-Pad2)
- T1 pad 3: Net-(C23-Pad2) -> Net-(R37-Pad1)
- T2 pad 1: Net-(R38-Pad1) -> Net-(R42-Pad2)
- T2 pad 2: Net-(R42-Pad2) -> Net-(C24-Pad1)
- T2 pad 3: Net-(C24-Pad1) -> Net-(R38-Pad1)
- T3 pad 2: Net-(C19-Pad1) -> Net-(C23-Pad2)
- T3 pad 3: Net-(C23-Pad2) -> Net-(C19-Pad1)
- T4 pad 1: Net-(C20-Pad2) -> Net-(R44-Pad2)
- T4 pad 2: Net-(R44-Pad2) -> Net-(C24-Pad1)
- T4 pad 3: Net-(C24-Pad1) -> Net-(C20-Pad2)
Routing:
- net GND: track 1049.1 -> 1158.3 mm
- net Net-(R37-Pad1): track 31.0 -> 80.4 mm
- net Net-(R38-Pad1): track 50.0 -> 99.1 mm
- net Net-(C19-Pad1): track 56.6 -> 13.4 mm
- net Net-(Q17-Pad1): track 65.8 -> 27.6 mm
- net Net-(Q16-Pad1): track 42.0 -> 73.3 mm
- net Net-(C20-Pad2): track 51.0 -> 33.1 mm
- net Net-(R42-Pad2): track 21.0 -> 4.38 mm
- net Net-(R44-Pad2): track 20.9 -> 4.38 mm
- net Net-(C23-Pad2): track 149.4 -> 154.5 mm
- net Net-(R41-Pad2): track 0.00 -> 3.85 mm
- net Net-(R43-Pad2): track 0.00 -> 3.85 mm
- net Net-(C24-Pad1): track 195.3 -> 191.9 mm
- net Net-(C17-Pad1): track 151.6 -> 152.9 mm
