File: LeachAmp_kicad/LeachAmp_kicad.sch (KiCad schematic (older format))
At the start: 119 parts, among them J1 Conn_01x12_Female, J2 Conn_01x04_Female, J3 Conn_01x03_Female, J4 Conn_01x03_Female, Q1 BC546, Q10 MPSA06, Q11 MPSA56, Q12 BF470, Q13 BF469, Q14 BF469, Q15 BF470, Q16 MJE15030, Q17 MJE15031, Q2 BC546, Q3 BC556, Q4 BC556, Q5 BC546, Q6 BC556, Q7 BD139, Q8 BC556, Q9 BC546, T1 MJL3281, T2 MJL3201, T3 MJL3281, T4 MJL3201

Commit message: oprava tranzistoru
Parts:
- Q15: symbol Transistor_BJT:MPSA92 -> Transistor_BJT:2SB631
- Q16: symbol Transistor_BJT:MPSA42 -> Transistor_BJT:BCX56
- Q17, T2, T4: symbol Transistor_BJT:MPSA92 -> Transistor_BJT:PBSS301PZ
- T1, T3: symbol Transistor_BJT:2N3055 -> Transistor_BJT:BCX56
- gave numbers to parts that had none: 1
Connections:
- net at R36.2, R42.1, R44.1: now also Q17.3 (E); no longer Q17.1 (E)
- net at R42.2: now also T2.1 (B); no longer T2.2 (B)
- net at R44.2: now also T4.1 (B); no longer T4.2 (B)
- net at C11.1, C12.1, D8.2 (A)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: now also Q15.3 (B); no longer Q15.2 (B)
- net at Q15.1 (E), R35.2: now also Q17.1 (B); no longer Q17.2 (B)
- net at C24.1, C27.2, D12.1 (K)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: now also Q15.2 (C), Q17.2 (C), Q17.4 (C), T2.2 (C), T2.4 (C), T4.2 (C), T4.4 (C); no longer Q15.3 (C), Q17.3 (C), T2.3 (C), T4.3 (C)
- net at Q14.1 (E), R34.1: now also Q16.1 (B); no longer Q16.2 (B)
- net at C23.2, C6.2, D11.2 (A)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: now also Q16.2 (C), T1.2 (C), T3.2 (C); no longer Q16.3 (C), T1.3 (C), T3.3 (C)
- net at R36.1, R41.1, R43.1: now also Q16.3 (E); no longer Q16.1 (E)
- net at R38.1, R46.1: now also T2.3 (E); no longer T2.1 (E)
- net at C20.2, R40.2, R48.1: now also T4.3 (E); no longer T4.1 (E)
- net at C19.1, R39.1, R47.2: now also T3.3 (E); no longer T3.2 (E)
- net at R37.1, R45.2: now also T1.3 (E); no longer T1.2 (E)
Changed lines of the file:
@@
 	7950 7500 7950 7300
 $Comp
-L Transistor_BJT:MPSA92 Q15
+L Transistor_BJT:2SB631 Q15
 U 1 1 5FE92B38
 P 9150 6450
@@
 $EndComp
 $Comp
-L Transistor_BJT:MPSA42 Q16
+L Transistor_BJT:BCX56 Q16
 U 1 1 5FEB116D
 P 9850 3950
@@
 $EndComp
 $Comp
-L Transistor_BJT:MPSA92 Q17
+L Transistor_BJT:PBSS301PZ Q17
 U 1 1 5FEA4EFE
 P 9850 6450
@@
 	6200 5500 6400 5500
 $Comp
-L Transistor_BJT:2N3055 T1
+L Transistor_BJT:BCX56 T1
 U 1 1 600AD28A
 P 10750 3950
@@
 	10550 3950 10400 3950
 $Comp
-L Transistor_BJT:2N3055 T3
+L Transistor_BJT:BCX56 T3
 U 1 1 600E7B95
 P 11650 3950
@@
 	11450 3950 11100 3950
 $Comp
-L Transistor_BJT:MPSA92 T2
+L Transistor_BJT:PBSS301PZ T2
 U 1 1 60106461
 P 10750 6450
@@
 $EndComp
 $Comp
-L Transistor_BJT:MPSA92 T4
+L Transistor_BJT:PBSS301PZ T4
 U 1 1 601226DD
 P 11650 6450
@@
 	6350 5050 6400 5050
 $Comp
-L Connector:Conn_01x03_Female J?
+L Connector:Conn_01x03_Female J5
 U 1 1 6004D92D
 P 6350 9250
-F 0 "J?" H 6242 8925 50  0000 C CNN
+F 0 "J5" H 6242 8925 50  0000 C CNN
 F 1 "Conn_01x03_Female" V 6400 9250 50  0000 C CNN
 F 2 "Connector_Molex:Molex_KK-254_AE-6410-03A_1x03_P2.54mm_Vertical" H 6350 9250 50  0001 C CNN
