File: LeachAmp_kicad/LeachAmp_kicad.sch (KiCad schematic (older format))
At the start: 119 parts, among them J1 Conn_01x12_Female, J2 Conn_01x04_Female, J3 Conn_01x03_Female, J4 Conn_01x03_Female, Q1 BC546, Q10 MPSA06, Q11 MPSA56, Q12 BF470, Q13 BF469, Q14 BF469, Q15 BF470, Q16 MJE15030, Q17 MJE15031, Q2 BC546, Q3 BC556, Q4 BC556, Q5 BC546, Q6 BC556, Q7 BD139, Q8 BC556, Q9 BC546, T1 MJL3281, T2 MJL3201, T3 MJL3281, T4 MJL3201

Commit message: nove_rozmery_soucastek
Nové rozměry součástek hlavně u kondenzátorů
Parts:
- C12, C17, C18, C7: footprint Capacitor_THT:C_Rect_L7.2mm_W3.5mm_P5.00mm_FKS2_FKP2_MKS2_MKP2 -> Capacitor_THT:C_Rect_L10.0mm_W2.5mm_P7.50mm_MKS4
- C13, C14, C4, C5: footprint Capacitor_THT:CP_Radial_D12.5mm_P7.50mm -> Capacitor_THT:CP_Radial_D10.0mm_P5.00mm
- C15, C16, C2, C23, C24, C27, C3, C6: footprint Capacitor_THT:C_Rect_L10.3mm_W5.7mm_P7.50mm_MKS4 -> Capacitor_THT:C_Rect_L10.0mm_W2.5mm_P7.50mm_MKS4
- C19, C20: footprint Capacitor_THT:C_Rect_L7.2mm_W3.5mm_P5.00mm_FKS2_FKP2_MKS2_MKP2 -> Capacitor_THT:C_Rect_L7.2mm_W2.5mm_P5.00mm_FKS2_FKP2_MKS2_MKP2
- Q15: symbol Transistor_BJT:MPSA92 -> Transistor_BJT:2SB631
- Q16: symbol Transistor_BJT:MPSA42 -> Transistor_BJT:BCX56
- Q17, T2, T4: symbol Transistor_BJT:MPSA92 -> Transistor_BJT:PBSS301PZ
- T1, T3: symbol Transistor_BJT:2N3055 -> Transistor_BJT:BCX56
- gave numbers to parts that had none: 1
Connections:
- net at R36.2, R42.1, R44.1: now also Q17.3 (E); no longer Q17.1 (E)
- net at R42.2: now also T2.1 (B); no longer T2.2 (B)
- net at R44.2: now also T4.1 (B); no longer T4.2 (B)
- net at C11.1, C12.1, D8.2 (A)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: now also Q15.3 (B); no longer Q15.2 (B)
- net at Q15.1 (E), R35.2: now also Q17.1 (B); no longer Q17.2 (B)
- net at C24.1, C27.2, D12.1 (K)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: now also Q15.2 (C), Q17.2 (C), Q17.4 (C), T2.2 (C), T2.4 (C), T4.2 (C), T4.4 (C); no longer Q15.3 (C), Q17.3 (C), T2.3 (C), T4.3 (C)
- net at Q14.1 (E), R34.1: now also Q16.1 (B); no longer Q16.2 (B)
- net at C23.2, C6.2, D11.2 (A)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: now also Q16.2 (C), T1.2 (C), T3.2 (C); no longer Q16.3 (C), T1.3 (C), T3.3 (C)
- net at R36.1, R41.1, R43.1: now also Q16.3 (E); no longer Q16.1 (E)
- net at R38.1, R46.1: now also T2.3 (E); no longer T2.1 (E)
- net at C20.2, R40.2, R48.1: now also T4.3 (E); no longer T4.1 (E)
- net at C19.1, R39.1, R47.2: now also T3.3 (E); no longer T3.2 (E)
- net at R37.1, R45.2: now also T1.3 (E); no longer T1.2 (E)
Changed lines of the file:
@@
 F 0 "C2" V 5150 3300 50  0000 L CNN
 F 1 "100n/100V film" V 5250 3200 50  0000 L CNN
-F 2 "Capacitor_THT:C_Rect_L10.3mm_W5.7mm_P7.50mm_MKS4" H 5138 3300 50  0001 C CNN
+F 2 "Capacitor_THT:C_Rect_L10.0mm_W2.5mm_P7.50mm_MKS4" H 5138 3300 50  0001 C CNN
 F 3 "~" H 5100 3450 50  0001 C CNN
 	1    5100 3450
@@
 F 0 "C12" V 6650 5350 50  0000 L CNN
 F 1 "100n/50V film" V 6550 5000 50  0000 L CNN
-F 2 "Capacitor_THT:C_Rect_L7.2mm_W3.5mm_P5.00mm_FKS2_FKP2_MKS2_MKP2" H 6738 5100 50  0001 C CNN
+F 2 "Capacitor_THT:C_Rect_L10.0mm_W2.5mm_P7.50mm_MKS4" H 6738 5100 50  0001 C CNN
 F 3 "~" H 6700 5250 50  0001 C CNN
 	1    6700 5250
@@
 F 0 "C4" V 5500 3500 50  0000 L CNN
 F 1 "100u/63V" V 5600 3250 50  0000 L CNN
-F 2 "Capacitor_THT:CP_Radial_D12.5mm_P7.50mm" H 5488 3300 50  0001 C CNN
+F 2 "Capacitor_THT:CP_Radial_D10.0mm_P5.00mm" H 5488 3300 50  0001 C CNN
 F 3 "~" H 5450 3450 50  0001 C CNN
 	1    5450 3450
@@
 F 0 "C3" V 4550 7500 50  0000 L CNN
 F 1 "100n/100V film" V 4650 7150 50  0000 L CNN
-F 2 "Capacitor_THT:C_Rect_L10.3mm_W5.7mm_P7.50mm_MKS4" H 4538 7300 50  0001 C CNN
+F 2 "Capacitor_THT:C_Rect_L10.0mm_W2.5mm_P7.50mm_MKS4" H 4538 7300 50  0001 C CNN
 F 3 "~" H 4500 7450 50  0001 C CNN
 	1    4500 7450
@@
 F 0 "C5" V 4900 7500 50  0000 L CNN
 F 1 "100u/63V" V 5000 7300 50  0000 L CNN
-F 2 "Capacitor_THT:CP_Radial_D12.5mm_P7.50mm" H 4888 7300 50  0001 C CNN
+F 2 "Capacitor_THT:CP_Radial_D10.0mm_P5.00mm" H 4888 7300 50  0001 C CNN
 F 3 "~" H 4850 7450 50  0001 C CNN
 	1    4850 7450
@@
 F 0 "C7" V 5400 6100 50  0000 L CNN
 F 1 "100n/50V film" V 5500 6000 50  0000 L CNN
-F 2 "Capacitor_THT:C_Rect_L7.2mm_W3.5mm_P5.00mm_FKS2_FKP2_MKS2_MKP2" H 5388 6100 50  0001 C CNN
+F 2 "Capacitor_THT:C_Rect_L10.0mm_W2.5mm_P7.50mm_MKS4" H 5388 6100 50  0001 C CNN
 F 3 "~" H 5350 6250 50  0001 C CNN
 	1    5350 6250
@@
 F 0 "C14" H 6700 7700 50  0000 L CNN
 F 1 "100u/63V" H 6600 7500 50  0000 L CNN
-F 2 "Capacitor_THT:CP_Radial_D12.5mm_P7.50mm" H 6888 7650 50  0001 C CNN
+F 2 "Capacitor_THT:CP_Radial_D10.0mm_P5.00mm" H 6888 7650 50  0001 C CNN
 F 3 "~" H 6850 7800 50  0001 C CNN
 	1    6850 7800
@@
 F 0 "C16" H 7250 7700 50  0000 L CNN
 F 1 "100n/100V film" H 7100 7500 50  0000 L CNN
-F 2 "Capacitor_THT:C_Rect_L10.3mm_W5.7mm_P7.50mm_MKS4" H 7288 7650 50  0001 C CNN
+F 2 "Capacitor_THT:C_Rect_L10.0mm_W2.5mm_P7.50mm_MKS4" H 7288 7650 50  0001 C CNN
 F 3 "~" H 7250 7800 50  0001 C CNN
 	1    7250 7800
@@
 F 0 "C15" V 7300 2300 50  0000 L CNN
 F 1 "100n/100V" V 7400 2250 50  0000 L CNN
-F 2 "Capacitor_THT:C_Rect_L10.3mm_W5.7mm_P7.50mm_MKS4" H 7288 2350 50  0001 C CNN
+F 2 "Capacitor_THT:C_Rect_L10.0mm_W2.5mm_P7.50mm_MKS4" H 7288 2350 50  0001 C CNN
 F 3 "~" H 7250 2500 50  0001 C CNN
 	1    7250 2500
@@
 F 0 "C17" V 7900 4900 50  0000 L CNN
 F 1 "100n/50V film" V 8100 4700 50  0000 L CNN
-F 2 "Capacitor_THT:C_Rect_L7.2mm_W3.5mm_P5.00mm_FKS2_FKP2_MKS2_MKP2" H 7988 4950 50  0001 C CNN
+F 2 "Capacitor_THT:C_Rect_L10.0mm_W2.5mm_P7.50mm_MKS4" H 7988 4950 50  0001 C CNN
 F 3 "~" H 7950 5100 50  0001 C CNN
 	1    7950 5100
@@
 F 0 "C18" V 7900 5550 50  0000 L CNN
 F 1 "100n/50V film" V 8100 5350 50  0000 L CNN
-F 2 "Capacitor_THT:C_Rect_L7.2mm_W3.5mm_P5.00mm_FKS2_FKP2_MKS2_MKP2" H 7988 5350 50  0001 C CNN
+F 2 "Capacitor_THT:C_Rect_L10.0mm_W2.5mm_P7.50mm_MKS4" H 7988 5350 50  0001 C CNN
 F 3 "~" H 7950 5500 50  0001 C CNN
 	1    7950 5500
@@
 	7950 7500 7950 7300
 $Comp
-L Transistor_BJT:MPSA92 Q15
+L Transistor_BJT:2SB631 Q15
 U 1 1 5FE92B38
 P 9150 6450
@@
 $EndComp
 $Comp
-L Transistor_BJT:MPSA42 Q16
+L Transistor_BJT:BCX56 Q16
 U 1 1 5FEB116D
 P 9850 3950
@@
 F 0 "C19" V 11300 4750 50  0000 L CNN
 F 1 "10n/50V film" V 11400 4500 50  0000 L CNN
-F 2 "Capacitor_THT:C_Rect_L7.2mm_W3.5mm_P5.00mm_FKS2_FKP2_MKS2_MKP2" H 11288 4550 50  0001 C CNN
+F 2 "Capacitor_THT:C_Rect_L7.2mm_W2.5mm_P5.00mm_FKS2_FKP2_MKS2_MKP2" H 11288 4550 50  0001 C CNN
 F 3 "~" H 11250 4700 50  0001 C CNN
 	1    11250 4700
@@
 F 0 "C20" V 11350 5450 50  0000 L CNN
 F 1 "10n/50V film" V 11450 5350 50  0000 L CNN
-F 2 "Capacitor_THT:C_Rect_L7.2mm_W3.5mm_P5.00mm_FKS2_FKP2_MKS2_MKP2" H 11338 5500 50  0001 C CNN
+F 2 "Capacitor_THT:C_Rect_L7.2mm_W2.5mm_P5.00mm_FKS2_FKP2_MKS2_MKP2" H 11338 5500 50  0001 C CNN
 F 3 "~" H 11300 5650 50  0001 C CNN
 	1    11300 5650
@@
 F 0 "C13" V 6900 2300 50  0000 L CNN
 F 1 "100u/63V" V 7000 2300 50  0000 L CNN
-F 2 "Capacitor_THT:CP_Radial_D12.5mm_P7.50mm" H 6888 2350 50  0001 C CNN
+F 2 "Capacitor_THT:CP_Radial_D10.0mm_P5.00mm" H 6888 2350 50  0001 C CNN
 F 3 "~" H 6850 2500 50  0001 C CNN
 	1    6850 2500
@@
 $EndComp
 $Comp
-L Transistor_BJT:MPSA92 Q17
+L Transistor_BJT:PBSS301PZ Q17
 U 1 1 5FEA4EFE
 P 9850 6450
@@
 F 0 "C24" V 12150 7550 50  0000 L CNN
 F 1 "100n/100V film" V 12250 7450 50  0000 L CNN
-F 2 "Capacitor_THT:C_Rect_L10.3mm_W5.7mm_P7.50mm_MKS4" H 12138 7600 50  0001 C CNN
+F 2 "Capacitor_THT:C_Rect_L10.0mm_W2.5mm_P7.50mm_MKS4" H 12138 7600 50  0001 C CNN
 F 3 "~" H 12100 7750 50  0001 C CNN
 	1    12100 7750
@@
 F 0 "C23" V 12100 2350 50  0000 L CNN
 F 1 "100n/100V film" V 12200 2250 50  0000 L CNN
-F 2 "Capacitor_THT:C_Rect_L10.3mm_W5.7mm_P7.50mm_MKS4" H 12088 2400 50  0001 C CNN
+F 2 "Capacitor_THT:C_Rect_L10.0mm_W2.5mm_P7.50mm_MKS4" H 12088 2400 50  0001 C CNN
 F 3 "~" H 12050 2550 50  0001 C CNN
 	1    12050 2550
@@
 F 0 "C6" V 11350 2350 50  0000 L CNN
 F 1 "100n/100V film" V 11450 2250 50  0000 L CNN
-F 2 "Capacitor_THT:C_Rect_L10.3mm_W5.7mm_P7.50mm_MKS4" H 11338 2400 50  0001 C CNN
+F 2 "Capacitor_THT:C_Rect_L10.0mm_W2.5mm_P7.50mm_MKS4" H 11338 2400 50  0001 C CNN
 F 3 "~" H 11300 2550 50  0001 C CNN
 	1    11300 2550
@@
 F 0 "C27" V 11350 7550 50  0000 L CNN
 F 1 "100n/100V film" V 11450 7450 50  0000 L CNN
-F 2 "Capacitor_THT:C_Rect_L10.3mm_W5.7mm_P7.50mm_MKS4" H 11338 7600 50  0001 C CNN
+F 2 "Capacitor_THT:C_Rect_L10.0mm_W2.5mm_P7.50mm_MKS4" H 11338 7600 50  0001 C CNN
 F 3 "~" H 11300 7750 50  0001 C CNN
 	1    11300 7750
@@
 	6200 5500 6400 5500
 $Comp
-L Transistor_BJT:2N3055 T1
+L Transistor_BJT:BCX56 T1
 U 1 1 600AD28A
 P 10750 3950
@@
 	10550 3950 10400 3950
 $Comp
-L Transistor_BJT:2N3055 T3
+L Transistor_BJT:BCX56 T3
 U 1 1 600E7B95
 P 11650 3950
@@
 	11450 3950 11100 3950
 $Comp
-L Transistor_BJT:MPSA92 T2
+L Transistor_BJT:PBSS301PZ T2
 U 1 1 60106461
 P 10750 6450
@@
 $EndComp
 $Comp
-L Transistor_BJT:MPSA92 T4
+L Transistor_BJT:PBSS301PZ T4
 U 1 1 601226DD
 P 11650 6450
@@
 	6350 5050 6400 5050
 $Comp
-L Connector:Conn_01x03_Female J?
+L Connector:Conn_01x03_Female J5
 U 1 1 6004D92D
 P 6350 9250
-F 0 "J?" H 6242 8925 50  0000 C CNN
+F 0 "J5" H 6242 8925 50  0000 C CNN
 F 1 "Conn_01x03_Female" V 6400 9250 50  0000 C CNN
 F 2 "Connector_Molex:Molex_KK-254_AE-6410-03A_1x03_P2.54mm_Vertical" H 6350 9250 50  0001 C CNN
